Commit message: Add files via upload

File: streetdrone_model/sd_description/urdf/sd_twizy.urdf.xacro (robot description, xacro)
@@ -1,5 +1,5 @@
 <?xml version="1.0"?>
 <!--
-Copyright (c) 2020 StreetDrone Limited
+Copyright (c) 2019 StreetDrone Limited
 Author:  Efimia Panagiotaki
 All rights reserved
@@ -12,5 +12,4 @@
   <xacro:include filename="$(find sd_description)/urdf/wheels/sd_twizy_suspension.urdf.xacro" />
   <xacro:include filename="$(find sd_description)/urdf/sensors/VLP-16.urdf.xacro"/>
-  <xacro:include filename="$(find sd_description)/urdf/sensors/cameras.urdf.xacro"/>
   <!-- *************** -->
   <!-- Robots Elements -->
@@ -22,31 +21,7 @@
   <xacro:FR_wheel/>
   <!-- Sensors -->
-  <xacro:VLP-16  parent="chassis" name="velodyne" topic="/points_raw" hz="10" samples="1875">
+  <xacro:VLP-16  parent="chassis" name="velodyne" topic="/velodyne_points" hz="10" samples="1875">
     <origin xyz="-0.681 0 1.445" rpy="0 -${1.5*M_PI/180.0} 0"/>
   </xacro:VLP-16>
-  <xacro:blackfly_camera frlr_prefix="front" lrc_prefix="left">
-    <origin xyz="-0.04 0.12 1.3" rpy="0 0.087 0"/>
-  </xacro:blackfly_camera>
-  <xacro:blackfly_camera frlr_prefix="front" lrc_prefix="right">
-    <origin xyz="-0.04 -0.12 1.3" rpy="0 0.087 0"/>
-  </xacro:blackfly_camera>
-  <xacro:blackfly_camera frlr_prefix="front" lrc_prefix="center">
-    <origin xyz="-0.04 0 1.3" rpy="0 0.087 0"/>
-  </xacro:blackfly_camera>
-  <xacro:blackfly_camera frlr_prefix="rear" lrc_prefix="center">
-    <origin xyz="-1.26 0 1.28" rpy="0 0.2618 3.14"/>
-  </xacro:blackfly_camera>
-  <xacro:blackfly_camera frlr_prefix="right" lrc_prefix="forward">
-    <origin xyz="-0.95 -0.42 1.2" rpy="0 0.244 -1.12"/>
-  </xacro:blackfly_camera>
-  <xacro:blackfly_camera frlr_prefix="right" lrc_prefix="rearward">
-    <origin xyz="-1.05 -0.42 1.2" rpy="0 0.244 -2.18"/>
-  </xacro:blackfly_camera>
-  <xacro:blackfly_camera frlr_prefix="left" lrc_prefix="forward">
-    <origin xyz="-0.95 0.4 1.2" rpy="0 0.2967 1.12"/>
-  </xacro:blackfly_camera>
-  <xacro:blackfly_camera frlr_prefix="left" lrc_prefix="rearward">
-    <origin xyz="-1.05 0.39 1.2" rpy="0 0.2967 2.18"/>
-  </xacro:blackfly_camera>
   <gazebo>
     <plugin name="sd_control" filename="libSdControlPlugin.so">

File: streetdrone_model/sd_description/urdf/sensors/VLP-16.urdf.xacro (robot description, xacro)
@@ -2,5 +2,5 @@
 <robot xmlns:xacro="http://www.ros.org/wiki/xacro" name="VLP-16">
     <xacro:property name="M_PI" value="3.1415926535897931" />
-    <xacro:macro name="VLP-16" params="*origin parent:=base_link name:=velodyne topic:=/points_raw hz:=10 lasers:=16 samples:=1875 collision_range:=0.3 min_range:=0.9 max_range:=130.0 noise:=0.008 min_angle:=-${M_PI} max_angle:=${M_PI} gpu:=false">
+    <xacro:macro name="VLP-16" params="*origin parent:=base_link name:=velodyne topic:=/velodyne_points hz:=10 lasers:=16 samples:=1875 collision_range:=0.3 min_range:=0.9 max_range:=130.0 noise:=0.008 min_angle:=-${M_PI} max_angle:=${M_PI} gpu:=false">
         <joint name="${name}_base_mount_joint" type="fixed">
             <xacro:insert_block name="origin" />

File: streetdrone_model/sd_description/urdf/wheels/sd_twizy_suspension.urdf.xacro (robot description, xacro)
@@ -1,5 +1,5 @@
 <?xml version="1.0"?>
 <!--
-Copyright (c) 2020 StreetDrone Limited
+Copyright (c) 2019 StreetDrone Limited
 Author:  Efimia Panagiotaki
 All rights reserved
