Commit message: Add files via upload

File: streetdrone_model/sd_description/urdf/sensors/VLP-16.urdf.xacro (robot description, xacro)
@@ -2,5 +2,5 @@
 <robot xmlns:xacro="http://www.ros.org/wiki/xacro" name="VLP-16">
     <xacro:property name="M_PI" value="3.1415926535897931" />
-    <xacro:macro name="VLP-16" params="*origin parent:=base_link name:=velodyne topic:=/points_raw hz:=10 lasers:=16 samples:=1875 collision_range:=0.3 min_range:=0.9 max_range:=130.0 noise:=0.008 min_angle:=-${M_PI} max_angle:=${M_PI} gpu:=false">
+    <xacro:macro name="VLP-16" params="*origin parent:=base_link name:=velodyne topic:=/points_raw hz:=15 lasers:=16 samples:=1875 collision_range:=0.3 min_range:=0.5 max_range:=10.0 noise:=0.008 min_angle:=-${M_PI} max_angle:=${M_PI} gpu:=true">
         <joint name="${name}_base_mount_joint" type="fixed">
             <xacro:insert_block name="origin" />
