Commit message: Add files via upload
updated twizy description files to include an imu simulation

File: streetdrone_model/sd_description/urdf/bases/sd_twizy_body.urdf.xacro (robot description, xacro)
@@ -22,4 +22,10 @@
       </visual>
     </link>
+<joint name="imu_joint" type="fixed">
+    <parent link="base_link"/>
+    <child link="imu_link"/>
+    <origin xyz="0 0 0" rpy="0 0 0"/>
+  </joint>
+  <link name="imu_link"/>
     <joint name="chassis_joint" type="fixed">
       <origin xyz="${wheelbase / 2} 0 0" rpy="0 0 0"/>

File: streetdrone_model/sd_description/urdf/sd_twizy.urdf.xacro (robot description, xacro)
@@ -62,3 +62,18 @@
     </plugin>
   </gazebo>
+ <gazebo reference="imu_link">
+    <gravity>true</gravity>
+    <sensor name="imu_sensor" type="imu">
+      <always_on>true</always_on>
+      <update_rate>100</update_rate>
+      <visualize>true</visualize>
+      <plugin filename="libgazebo_ros_imu_sensor.so" name="imu_plugin">
+        <topicName>imu</topicName>
+        <bodyName>imu_link</bodyName>
+        <updateRateHZ>10.0</updateRateHZ>
+        <gaussianNoise>0.0</gaussianNoise>
+        <frameName>imu_link</frameName>
+      </plugin>
+    </sensor>
+  </gazebo>
 </robot>

File: streetdrone_model/sd_description/urdf/sensors/VLP-16.urdf.xacro (robot description, xacro)
@@ -2,5 +2,5 @@
 <robot xmlns:xacro="http://www.ros.org/wiki/xacro" name="VLP-16">
     <xacro:property name="M_PI" value="3.1415926535897931" />
-    <xacro:macro name="VLP-16" params="*origin parent:=base_link name:=velodyne topic:=/velodyne_points hz:=10 lasers:=16 samples:=1875 collision_range:=0.3 min_range:=0.9 max_range:=130.0 noise:=0.008 min_angle:=-${M_PI} max_angle:=${M_PI} gpu:=false">
+    <xacro:macro name="VLP-16" params="*origin parent:=base_link name:=velodyne topic:=/velodyne_points hz:=10 lasers:=16 samples:=1875 collision_range:=0.3 min_range:=0.9 max_range:=130.0 noise:=0.008 min_angle:=-${M_PI} max_angle:=${M_PI} gpu:=true">
         <joint name="${name}_base_mount_joint" type="fixed">
             <xacro:insert_block name="origin" />
